Commit message: Initialize challenge solution
* fix mismatch arm urdf for hab suction
* change `rigid_obj_dir` to be compatible with challenge env

File: habitat_extensions/assets/robots/hab_fetch/robots/hab_fetch_arm_v2.urdf (robot description, URDF)
Before this commit: robot fetch, 10 links, 9 joints
Links:
- link gripper_link: geometry collision box size=0.04 0.04 0.18
Joints:
- joint gripper_axis: origin xyz=0.16645 0 0 rpy=0 0 0 -> xyz=0.16645 0 0 rpy=0 1.56 0

Commit message: Update challenge solution

File: habitat_extensions/assets/robots/hab_fetch/robots/hab_fetch_arm_v2.urdf (robot description, URDF)
Before this commit: robot fetch, 10 links, 9 joints
Links:
- link base_link: geometry 
- link elbow_flex_link: geometry collision mesh filename=../meshes/elbow_flex_link_collision.obj
- link forearm_roll_link: geometry collision mesh filename=../meshes/forearm_roll_link_collision.obj
- link shoulder_lift_link: geometry collision mesh filename=../meshes/shoulder_lift_link_collision.obj
- link shoulder_pan_link: geometry 
- link suction_link: geometry collision box size=0.04 0.04 0.01
- link upperarm_roll_link: geometry collision mesh filename=../meshes/upperarm_roll_link_collision.obj
- link wrist_flex_link: geometry collision mesh filename=../meshes/wrist_flex_link_collision.obj
- link wrist_roll_link: geometry collision mesh filename=../meshes/wrist_roll_link_collision.obj
